File: retroclock-v1.1/retroclock-v1.1.kicad_sch (KiCad schematic)
At the start: 22 parts, among them J1 Hours, J2 Mins, J3 Secs, J4 Nixie YY2, J5 Nixie YY1, J6 Nixie MM2, J7 Nixie MM1, J8 Nixie DD2, J9 Nixie DD1

Commit message: finished routing, no errors
Parts:
- J4, J5, J6, J7, J8, J9: footprint Connector_PinHeader_1.27mm:PinHeader_2x05_P1.27mm_Vertical -> Connector_PinHeader_1.27mm:PinHeader_1x10_P1.27mm_Vertical
Changed lines of the file:
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@@
 			)
 		)
-		(property "Footprint" "Connector_PinHeader_1.27mm:PinHeader_2x05_P1.27mm_Vertical"
+		(property "Footprint" "Connector_PinHeader_1.27mm:PinHeader_1x10_P1.27mm_Vertical"
 			(at 219.71 167.64 0)
 			(effects
@@
 			)
 		)
-		(property "Footprint" "Connector_PinHeader_1.27mm:PinHeader_2x05_P1.27mm_Vertical"
+		(property "Footprint" "Connector_PinHeader_1.27mm:PinHeader_1x10_P1.27mm_Vertical"
 			(at 274.32 144.78 0)
 			(effects
@@
 			)
 		)
-		(property "Footprint" "Connector_PinHeader_1.27mm:PinHeader_2x05_P1.27mm_Vertical"
+		(property "Footprint" "Connector_PinHeader_1.27mm:PinHeader_1x10_P1.27mm_Vertical"
 			(at 275.59 106.68 0)
 			(effects
@@
 			)
 		)
-		(property "Footprint" "Connector_PinHeader_1.27mm:PinHeader_2x05_P1.27mm_Vertical"
+		(property "Footprint" "Connector_PinHeader_1.27mm:PinHeader_1x10_P1.27mm_Vertical"
 			(at 269.24 66.04 0)
 			(effects
@@
 			)
 		)
-		(property "Footprint" "Connector_PinHeader_1.27mm:PinHeader_2x05_P1.27mm_Vertical"
+		(property "Footprint" "Connector_PinHeader_1.27mm:PinHeader_1x10_P1.27mm_Vertical"
 			(at 175.26 124.46 0)
 			(effects
@@
 			)
 		)
-		(property "Footprint" "Connector_PinHeader_1.27mm:PinHeader_2x05_P1.27mm_Vertical"
+		(property "Footprint" "Connector_PinHeader_1.27mm:PinHeader_1x10_P1.27mm_Vertical"
 			(at 273.05 30.48 0)
 			(effects

Commit message: retroclock 1.1 sent to JLCPCB!
Parts:
- removed C1, C2, C3: C, Capacitor_THT:CP_Axial_L18.0mm_D6.5mm_P25.00mm_Horizontal, symbol Device:C
- removed HL1, HL2: ~, mjc_library:PLCC-44_THT-Socket, symbol mjc_library:HL5122
- removed J1: Hours, Connector_PinHeader_1.27mm:PinHeader_1x02_P1.27mm_Vertical, symbol Connector:Conn_01x02_Pin
- removed J2: Mins, Connector_PinHeader_1.27mm:PinHeader_1x02_P1.27mm_Vertical, symbol Connector:Conn_01x02_Pin
- removed J3: Secs, Connector_PinHeader_1.27mm:PinHeader_1x02_P1.27mm_Vertical, symbol Connector:Conn_01x02_Pin
- removed J4: Nixie YY2, Connector_PinHeader_1.27mm:PinHeader_1x10_P1.27mm_Vertical, symbol Connector:Conn_01x10_Pin
- removed J5: Nixie YY1, Connector_PinHeader_1.27mm:PinHeader_1x10_P1.27mm_Vertical, symbol Connector:Conn_01x10_Pin
- removed J6: Nixie MM2, Connector_PinHeader_1.27mm:PinHeader_1x10_P1.27mm_Vertical, symbol Connector:Conn_01x10_Pin
- removed J7: Nixie MM1, Connector_PinHeader_1.27mm:PinHeader_1x10_P1.27mm_Vertical, symbol Connector:Conn_01x10_Pin
- removed J8: Nixie DD2, Connector_PinHeader_1.27mm:PinHeader_1x10_P1.27mm_Vertical, symbol Connector:Conn_01x10_Pin
- removed J9: Nixie DD1, Connector_PinHeader_1.27mm:PinHeader_1x10_P1.27mm_Vertical, symbol Connector:Conn_01x10_Pin
- removed R1, R2, R3, R4, R5, R6: R, Resistor_THT:R_Axial_DIN0207_L6.3mm_D2.5mm_P7.62mm_Horizontal, symbol Device:R
- added C10, C11: 100nF, Capacitor_THT:C_Disc_D3.4mm_W2.1mm_P2.50mm, symbol Device:C
- added C12: 68uF, Capacitor_THT:CP_Radial_D8.0mm_P3.80mm, symbol Device:C_Polarized
- added C13: 100uF, Capacitor_THT:CP_Radial_D10.0mm_P5.00mm, symbol Device:C_Polarized
- added C14: 100nF, Capacitor_THT:C_Rect_L18.0mm_W7.0mm_P15.00mm_FKS3_FKP3, symbol Device:C
- added C15, C16: 10uF, Capacitor_THT:CP_Radial_D8.0mm_P3.80mm, symbol Device:C_Polarized
- added C6, C8, C9: 100n, Capacitor_THT:C_Disc_D3.4mm_W2.1mm_P2.50mm, symbol Device:C
- added C7: 100n, Capacitor_SMD:C_1206_3216Metric_Pad1.33x1.80mm_HandSolder, symbol Device:C
- added D1, D4, D5: LED, LED_THT:LED_D3.0mm_Clear, symbol Device:LED
- added D3: RF01VM2S, Diode_THT:D_DO-15_P15.24mm_Horizontal, symbol Diode:RF01VM2S
- added H1, H2, H3, H4: MountingHole, MountingHole:MountingHole_2.2mm_M2_Pad, symbol Mechanical:MountingHole
- added J10: Serial DBG, Connector_PinHeader_2.54mm:PinHeader_1x03_P2.54mm_Vertical, symbol Connector:Conn_01x03_Pin
- added J12: Supply, Connector_Molex:Molex_KK-254_AE-6410-03A_1x03_P2.54mm_Vertical, symbol Connector:Conn_01x03_Pin
- added J13: 170V, Connector_Molex:Molex_KK-254_AE-6410-02A_1x02_P2.54mm_Vertical, symbol Connector:Conn_01x02_Pin
- added J14: ~, 01_mjc_library:Jumper 2.54 2x03, symbol mjc_library:Jumper 2x03
- added J15: 3v3 src, Connector_PinHeader_2.54mm:PinHeader_1x03_P2.54mm_Vertical, symbol Connector:Conn_01x03_Pin
- added L1: 100H, Inductor_THT:L_Radial_D10.0mm_P5.00mm_Neosid_SD12k_style3, symbol Device:L
- added MAX1: MAX1771, Package_SO:SOIC-8_3.9x4.9mm_P1.27mm, symbol mjc_library:MAX1771
- added Q1: ~, 01_mjc_library:MOSFET, symbol mjc_library:STD17NF25
- added R10: 1.2M, Resistor_THT:R_Axial_DIN0204_L3.6mm_D1.6mm_P7.62mm_Horizontal, symbol Device:R
- added R11: 10k, Resistor_THT:R_Axial_DIN0204_L3.6mm_D1.6mm_P7.62mm_Horizontal, symbol Device:R
- added R12, R9: 0.2, Resistor_THT:R_Axial_DIN0204_L3.6mm_D1.6mm_P7.62mm_Horizontal, symbol Device:R
- added R19, R20, R7: R, Resistor_THT:R_Axial_DIN0204_L3.6mm_D1.6mm_P7.62mm_Horizontal, symbol Device:R
- added U1: ~, 01_mjc_library:HT7333, symbol 01_mjc_library:HT7333
- ESP1: footprint mjc_library:ESP32 Header -> 01_mjc_library:ESP32 Header
- renumbered U1 to LVL1
Connections:
- net +12V: now also LVL1.16 (VDD), C11.1, C12.1, C15.1, C7.1, C9.2, J12.1 (Pin_1), J14.4, L1.1, MAX1.2 (V+), R19.2, U1.2 (Vi); no longer LVL1.18 (VDD)
- net +3V3: now also C6.2, J15.2 (Pin_2)
- net GND: now also C10.2, C11.2, C12.2, C13.2, C14.2, C15.2, C16.2, C6.1, C7.2, C8.2, C9.1, D1.1 (K), D4.1 (K), D5.1 (K), J10.3 (Pin_3), J12.3 (Pin_3), J13.1 (Pin_1), J14.6, MAX1.6 (AGND), MAX1.7 (GND), R11.2, R12.2, R9.2, U1.1 (GND)
- net NIX_CLK: now reaches LVL1.2 (AOUT)
- net SCL: now reaches ESP1.5 (SCL), LVL1.3 (AIN)
- net SCL: now also J10.1 (Pin_1)
- net NIX_OE: now reaches LVL1.4 (BOUT)
- net OE: now reaches ESP1.1 (G5), LVL1.5 (BIN)
- net NIX_DAT_IN: now reaches LVL1.6 (COUT)
- net SDA: now reaches ESP1.4 (SDA), LVL1.7 (CIN)
- net SDA: now also J10.2 (Pin_2), R7.1
- net AM_SEC: now reaches ESP1.8 (G21)
- net AM_HRS: now reaches ESP1.6 (G10)
- net AM_MIN: now reaches ESP1.7 (G20)
- net BOOST_EN: now reaches ESP1.10 (G1/A1_1)
- net BOOST_EN: now also J14.2
- net DCF_PON: now reaches ESP1.3 (G7)
- net DCF_DAT: now reaches ESP1.9 (G0/A1_0)
- new net: C8.1, J12.2 (Pin_2), J15.3 (Pin_3), R20.2
- new net: D3.2 (A), L1.2, Q1.2 (D)
- new net: D5.2 (A), R20.1
- new net: D4.2 (A), R19.1
- new net: D1.2 (A), R7.2
- new net: C16.1, J15.1 (Pin_1), U1.3 (Vo)
- new net: C10.1, MAX1.5 (REF)
- new net 170V: C13.1, C14.1, D3.1 (K), J13.2 (Pin_2), R10.1
- new net CS: MAX1.8 (CS), Q1.3 (S), R12.1, R9.1
- new net EXT: MAX1.1 (EXT), Q1.1 (G)
- new net FB: MAX1.3 (FB), R10.2, R11.1
- new net SHDN: J14.1, J14.3, J14.5, MAX1.4 (SHDN)
- no-connect marks 19 -> 12
Other:
- added sheet DCF77 (dcf77kicad_sch.kicad_sch)
- added sheet ammeter_driver (ammeter.kicad_sch)
- added sheet nixie driver (nixiedrv.kicad_sch)
- note added: "12V - 170V Step Up"
- note added: "170V"
- note added: "Ammeter driver"
- note added: "DCF77 receiver"
- note added: "EN"
- note added: "ESP32 Microprocessor"
- note added: "GND"
- note added: "Nixie driver"
- note added: "OFF"
- note added: "ON"
- note added: "Power supply"
- note added: "TTL to CMOS level shifter"
- note added: "Visual clock and oscill. probes"
- note added: "Vout"
- note added: "https://electronoobs.com/eng_circuitos_tut57.php"
- company: (none) -> jCAPS Corp.
- title: (none) -> Retro Clock
- moved on the sheet: ESP1, LVL1
